File: 2 - Clock/Clock.kicad_sch (KiCad schematic)
At the start: 69 parts, among them SW2 MODE, SW3 SPEED, SW4 STEP, SW5 BOOT SPEED, SW6 BOOT MODE, SW7 RESET FAST LSB, SW8 RESET FAST MSB, U1 74AC14, U10 74AC112, U11 74AC74, U12 LMC555, U13 74AC74, U14 74HC251, U15 74HC138, U16 74HC251, U17 74HC251, U3 74AC08, U4 74AC14, U5 74AC74, U6 74AC74, U7 74AC74, U8 74AC74, U9 74AC112, X1 14.7456MHz

Commit message: Clock card updated
Parts:
- SW5, SW6, SW7, SW8: footprint 0 - Library:Microswitch_4.7mm_spacing -> 0_Library:Microswitch_4.7mm_spacing
- U12: symbol 0 - Library:LMC555 -> 0_Library:LMC555
- X1: footprint 0 - Library:DIP-8-4_W7.62mm_Oscillator_Socket -> 0_Library:DIP-8-4_W7.62mm_Oscillator_Socket
