File: 3 - CPU and memory/3 - CPU and memory.kicad_pcb (KiCad board)
At the start: 2 copper layers, 100 x 100 mm, 48 parts, among them J1 EDGE, U1 74AC00, U10 74HC563, U2 74AC32, U3 74AC138, U4 Z84C0010, U5 SST39SF010, U6 AS6C4008, U7 74AC32, U8 74AC174, U9 74HC563

Commit message: Finished cleaning up the project
Parts:
- J1: footprint 0 - Library:BUS_XT -> 0_Library:BUS_XT_Proto
Routing:
- net GND: vias 4 -> 11
Other:
- outline, holes or cut-outs redrawn
- board text added: "ZedEighty Project - CPU and Memory Card - Rev 1.1 - Frédéric Segard - youtube.com/@microhobbyist"
- board text removed: "ZedEighty Project - CPU and Memory Card - Rev 1 - Frédéric Segard - youtube.com/@microhobbyist"
